File: pcb/car/car.kicad_pcb (KiCad board)
At the start: 2 copper layers, 60.3 x 63.5 mm, 9 parts

Commit message: feat: update pcb, update car code
Connections:
- ESP32_LEFT1 pad 1: +3.3V -> +3V3
- ESP32_RIGHT1 pad 9: /D33 -> +3.3V
- MD_RIGHT1 pad 5: GND -> /-
- MD_RIGHT1 pad 6: GND -> unconnected-(MD_RIGHT1-Pin_6-Pad6)
- SERVO1 pad 3: /D33 -> +3V3
- SERVO1 pad 5: GND -> /-
Routing:
- net +3V3: track 0.00 -> 58.8 mm
- net /D33: track 55.5 -> 0.00 mm
- net +3.3V: track 57.0 -> 42.2 mm
- net /+: track 49.8 -> 51.0 mm
Changed lines of the file:
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@@
 	(net 18 "/D34")
 	(net 19 "/D12")
-	(net 20 "/D33")
+	(net 20 "+3V3")
 	(net 21 "/D35")
 	(net 22 "/D32")
@@
 	(net 31 "/D2")
 	(net 32 "/D15")
+	(net 33 "/-")
+	(net 34 "unconnected-(MD_RIGHT1-Pin_6-Pad6)")
 	(footprint "Connector_PinSocket_2.54mm:PinSocket_1x01_P2.54mm_Vertical"
 		(layer "F.Cu")
@@
 			(layers "*.Cu" "*.Mask")
 			(remove_unused_layers no)
-			(net 5 "+3.3V")
+			(net 20 "+3V3")
 			(pinfunction "Pin_1")
 			(pintype "passive")
@@
 			(layers "*.Cu" "*.Mask")
 			(remove_unused_layers no)
-			(net 20 "/D33")
+			(net 20 "+3V3")
 			(pinfunction "Pin_3")
 			(pintype "passive")
@@
 			(layers "*.Cu" "*.Mask")
 			(remove_unused_layers no)
-			(net 1 "GND")
+			(net 33 "/-")
 			(pinfunction "Pin_5")
 			(pintype "passive")
@@
 			(layers "*.Cu" "*.Mask")
 			(remove_unused_layers no)
-			(net 20 "/D33")
+			(net 5 "+3.3V")
 			(pinfunction "Pin_9")
 			(pintype "passive")
@@
 			(layers "*.Cu" "*.Mask")
 			(remove_unused_layers no)
-			(net 1 "GND")
+			(net 33 "/-")
 			(pinfunction "Pin_5")
 			(pintype "passive")
@@
 			(layers "*.Cu" "*.Mask")
 			(remove_unused_layers no)
-			(net 1 "GND")
+			(net 34 "unconnected-(MD_RIGHT1-Pin_6-Pad6)")
 			(pinfunction "Pin_6")
 			(pintype "passive")
@@
 	)
 	(segment
-		(start 90.7 56)
-		(end 90.7 89.4)
+		(start 85 61.58)
+		(end 97.58 49)
 		(width 0.2)
 		(layer "F.Cu")
@@
 	)
 	(segment
-		(start 98.11 96.8)
-		(end 98.13 96.78)
+		(start 74.56 76.46)
+		(end 72.73 76.46)
 		(width 0.2)
 		(layer "F.Cu")
@@
 	)
 	(segment
-		(start 97.58 49.12)
-		(end 90.7 56)
+		(start 85 66)
+		(end 85 61.58)
 		(width 0.2)
 		(layer "F.Cu")
@@
 	)
 	(segment
-		(start 98.1 96.8)
-		(end 98.11 96.8)
+		(start 76.7 74.32)
+		(end 76.7 74.3)
 		(width 0.2)
 		(layer "F.Cu")
@@
 	)
 	(segment
-		(start 90.7 89.4)
-		(end 98.1 96.8)
+		(start 76.7 74.3)
+		(end 85 66)
 		(width 0.2)
 		(layer "F.Cu")
@@
 	)
 	(segment
+		(start 76.7 74.32)
+		(end 74.56 76.46)
+		(width 0.2)
+		(layer "F.Cu")
+		(net 5)
+	)
+	(segment
+		(start 97.58 49)
+		(end 97.58 49.12)
+		(width 0.2)
+		(layer "F.Cu")
+		(net 5)
+	)
+	(segment
 		(start 97.58 45.72)
-		(end 97.58 49.12)
+		(end 97.58 49)
 		(width 0.2)
 		(layer "F.Cu")
@@
 	)
 	(segment
-		(start 74.56 76.46)
-		(end 72.73 76.46)
+		(start 99.58 51.42)
+		(end 91 60)
 		(width 0.2)
 		(layer "F.Cu")
@@
 	)
 	(segment
-		(start 76.7 74.32)
-		(end 74.56 76.46)
-		(width 0.2)
-		(layer "F.Cu")
-		(net 20)
-	)
-	(segment
-		(start 76.7 50.6)
-		(end 76.7 74.32)
+		(start 98.11 96.8)
+		(end 98.13 96.78)
 		(width 0.2)
 		(layer "F.Cu")
@@
 	)
 	(segment
-		(start 98.7 43.9)
-		(end 83.4 43.9)
+		(start 91 89.5)
+		(end 91 89.7)
 		(width 0.2)
 		(layer "F.Cu")
@@
 	)
 	(segment
-		(start 83.4 43.9)
-		(end 76.7 50.6)
+		(start 98.1 96.8)
+		(end 98.11 96.8)
 		(width 0.2)
 		(layer "F.Cu")
@@
 	)
 	(segment
-		(start 99.58 44.78)
-		(end 98.7 43.9)
+		(start 99.58 45.72)
+		(end 99.58 51.42)
+		(width 0.2)
+		(layer "F.Cu")
+		(net 20)
+	)
+	(segment
+		(start 91 89.7)
+		(end 98.1 96.8)
+		(width 0.2)
+		(layer "F.Cu")
+		(net 20)
+	)
+	(segment
+		(start 91 60)
+		(end 91 89.7)
 		(width 0.2)
 		(layer "F.Cu")
@@
 	)
 	(segment
-		(start 123.2 86.566999)
-		(end 123.2 86.56)
+		(start 107 72.5)
+		(end 107 62.107215)
 		(width 1.5)
 		(layer "F.Cu")
@@
 	)
 	(segment
-		(start 101.58 45.72)
+		(start 123.2 86.56)
+		(end 121.06 86.56)
+		(width 1.5)
+		(layer "F.Cu")
+		(net 30)
+	)
+	(segment
+		(start 107 62.107215)
 		(end 101.58 56.687215)
 		(width 1.5)
@@
 	)
 	(segment
+		(start 121.06 86.56)
+		(end 107 72.5)
+		(width 1.5)
+		(layer "F.Cu")
+		(net 30)
+	)
+	(segment
 		(start 101.58 56.687215)
-		(end 106 61.107215)
-		(width 1.5)
-		(layer "F.Cu")
-		(net 30)
-	)
-	(segment
-		(start 106 69.366999)
-		(end 123.2 86.566999)
-		(width 1.5)
-		(layer "F.Cu")
-		(net 30)
-	)
-	(segment
-		(start 106 61.107215)
-		(end 106 69.366999)
+		(end 101.58 45.72)
 		(width 1.5)
 		(layer "F.Cu")
@@
 		(polygon
 			(pts
-				(xy 63.1 38.5) (xy 137.7 38.7) (xy 136.7 115.5) (xy 62.8 114.6) (xy 63.2 38.2)
+				(xy 135 109.5) (xy 135 39) (xy 64 40) (xy 64.5 110.5)
 			)
 		)
@@
 		(polygon
 			(pts
-				(xy 55.1 33.9) (xy 141.7 35.5) (xy 141.7 124) (xy 55.6 125.5)
-			)
-		)
+				(xy 55.5 35.5) (xy 145.5 34.5) (xy 142 122) (xy 54 121.5) (xy 55.5 36) (xy 55.5 35)
+			)
+		)
